File: Hardware/Maze Solver Robot/Maze Solver Robot.kicad_sch (KiCad schematic)
At the start: 0 parts

Commit message: Add final changes
Other:
- sheet Colour Light Sensing ports: added 3.3V, Green, Red; removed none
- sheet Communication ports: added 3.3V, B1, B2, LED1, LED2, LED3; removed none
- sheet Voltage Regulation ports: added 3.3V, Input (Battery?); removed none
Changed lines of the file:
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@@
 (kicad_sch (version 20211123) (generator eeschema)
   (paper "A4")
+  (junction (at 135.89 78.74) (diameter 0) (color 0 0 0 0)
+  )
+  (wire (pts (xy 135.89 78.74) (xy 135.89 122.555))
+    (stroke (width 0) (type default) (color 0 0 0 0))
+  )
+  (wire (pts (xy 125.73 78.74) (xy 135.89 78.74))
+    (stroke (width 0) (type default) (color 0 0 0 0))
+  )
+  (wire (pts (xy 125.095 122.555) (xy 135.89 122.555))
+    (stroke (width 0) (type default) (color 0 0 0 0))
+  )
+  (wire (pts (xy 135.89 78.74) (xy 142.24 78.74))
+    (stroke (width 0) (type default) (color 0 0 0 0))
+  )
   (sheet (at 65.405 48.26) (size 60.325 35.56) (fields_autoplaced)
     (stroke (width 0.1524) (type solid) (color 0 0 0 0))
@@
     (property "Sheet file" "communication.kicad_sch" (id 1) (at 65.405 84.4046 0)
       (effects (font (size 1.27 1.27)) (justify left top))
+    )
+    (pin "LED3" input (at 65.405 67.945 180)
+      (effects (font (size 1.27 1.27)) (justify left))
+    )
+    (pin "3.3V" input (at 125.73 78.74 0)
+      (effects (font (size 1.27 1.27)) (justify right))
+    )
+    (pin "B1" output (at 125.73 60.96 0)
+      (effects (font (size 1.27 1.27)) (justify right))
+    )
+    (pin "LED1" input (at 65.405 55.88 180)
+      (effects (font (size 1.27 1.27)) (justify left))
+    )
+    (pin "LED2" input (at 65.405 62.23 180)
+      (effects (font (size 1.27 1.27)) (justify left))
+    )
+    (pin "B2" output (at 125.73 69.85 0)
+      (effects (font (size 1.27 1.27)) (justify right))
     )
   )
@@
       (effects (font (size 1.27 1.27)) (justify left top))
     )
+    (pin "3.3V" input (at 142.24 78.74 180)
+      (effects (font (size 1.27 1.27)) (justify left))
+    )
+    (pin "Red" output (at 213.995 74.295 0)
+      (effects (font (size 1.27 1.27)) (justify right))
+    )
+    (pin "Green" output (at 213.995 67.31 0)
+      (effects (font (size 1.27 1.27)) (justify right))
+    )
   )
   (sheet (at 63.5 102.235) (size 61.595 34.925) (fields_autoplaced)
@@
     (property "Sheet file" "regulator.kicad_sch" (id 1) (at 63.5 137.7446 0)
       (effects (font (size 1.27 1.27)) (justify left top))
+    )
+    (pin "Input (Battery?)" input (at 63.5 113.03 180)
+      (effects (font (size 1.27 1.27)) (justify left))
+    )
+    (pin "3.3V" output (at 125.095 122.555 0)
+      (effects (font (size 1.27 1.27)) (justify right))
     )
   )
@@
     )
     (path "/3a52f112-cb97-43db-aaeb-20afe27664d7/2228514e-5299-4258-98b9-e9cdf9417856"
-      (reference "D?") (unit 1) (value "LED") (footprint "")
+      (reference "D?") (unit 1) (value "RED_LED") (footprint "")
     )
     (path "/3a52f112-cb97-43db-aaeb-20afe27664d7/5e31b75c-7539-48bc-9313-3ce6611e0cb9"
-      (reference "D?") (unit 1) (value "LED") (footprint "")
+      (reference "D?") (unit 1) (value "RED_LED") (footprint "")
     )
     (path "/3a52f112-cb97-43db-aaeb-20afe27664d7/68bd9244-ad41-43e6-b7c7-8d19b53f9a7a"
-      (reference "D?") (unit 1) (value "LED") (footprint "")
+      (reference "D?") (unit 1) (value "RED_LED") (footprint "")
     )
     (path "/e42b8b80-020c-4fee-b000-fd91abf3966d/292df1bb-c485-4816-83fb-4ace170c2ace"
       (reference "R?") (unit 1) (value "A1050") (footprint "OptoDevice:R_LDR_D6.4mm_P3.4mm_Vertical")
     )
+    (path "/3a52f112-cb97-43db-aaeb-20afe27664d7/628fb7ac-b2e6-4331-b594-4b06617cfdc7"
+      (reference "R?") (unit 1) (value "4.7k") (footprint "")
+    )
     (path "/3a52f112-cb97-43db-aaeb-20afe27664d7/7e6cef86-5304-43b4-a13e-c8be103e805f"
-      (reference "R?") (unit 1) (value "R_US") (footprint "")
+      (reference "R?") (unit 1) (value "33") (footprint "")
+    )
+    (path "/3a52f112-cb97-43db-aaeb-20afe27664d7/8f53dc68-99f9-4e88-8dd7-3e5c97f45722"
+      (reference "R?") (unit 1) (value "4.7k") (footprint "")
+    )
+    (path "/e42b8b80-020c-4fee-b000-fd91abf3966d/cd169261-b377-46f4-9b38-5619229b988a"
+      (reference "R?") (unit 1) (value "A1050") (footprint "OptoDevice:R_LDR_D6.4mm_P3.4mm_Vertical")
     )
     (path "/edf1a077-1088-4990-81c3-c25e6cc707f4/d4aea666-d9c1-4540-9e7d-952929720166"
@@
     )
     (path "/3a52f112-cb97-43db-aaeb-20afe27664d7/e71d8b01-ac1f-48ab-bc7c-1bec1ba57717"
-      (reference "R?") (unit 1) (value "R_US") (footprint "")
+      (reference "R?") (unit 1) (value "33") (footprint "")
     )
     (path "/edf1a077-1088-4990-81c3-c25e6cc707f4/fbb25297-cbc8-46f0-9efe-2186655c973e"
@@
     )
     (path "/3a52f112-cb97-43db-aaeb-20afe27664d7/fd073802-4dd7-4e04-9b9f-2340f5c8c06c"
-      (reference "R?") (unit 1) (value "R_US") (footprint "")
+      (reference "R?") (unit 1) (value "33") (footprint "")
     )
     (path "/e42b8b80-020c-4fee-b000-fd91abf3966d/211dafae-49cb-4e21-8b4b-ab2810e6e7a1"
-      (reference "RV?") (unit 1) (value "R_Potentiometer") (footprint "")
+      (reference "RV?") (unit 1) (value "R_Potentiometer_10K") (footprint "")
     )
     (path "/e42b8b80-020c-4fee-b000-fd91abf3966d/783e79f7-eca2-4551-a3b1-ad149f1459af"
-      (reference "RV?") (unit 1) (value "R_Potentiometer") (footprint "")
+      (reference "RV?") (unit 1) (value "R_Potentiometer_10K") (footprint "")
+    )
+    (path "/3a52f112-cb97-43db-aaeb-20afe27664d7/374334e0-4bfb-480f-8754-e799ef152f1f"
+      (reference "SW?") (unit 1) (value "SW_Push") (footprint "")
+    )
+    (path "/3a52f112-cb97-43db-aaeb-20afe27664d7/64abf69a-0e18-4187-9b02-701601313376"
+      (reference "SW?") (unit 1) (value "SW_Push") (footprint "")
+    )
+    (path "/edf1a077-1088-4990-81c3-c25e6cc707f4/6792a032-9256-487f-aa0b-8c689e242f4e"
+      (reference "U?") (unit 1) (value "LM317L_SOT-89") (footprint "Package_TO_SOT_SMD:SOT-89-3")
     )
     (path "/e42b8b80-020c-4fee-b000-fd91abf3966d/7aacff48-474b-4b07-91d1-3ae2bb730a02"
